File: maxpcb-ma22.kicad_pcb (KiCad board)
At the start: 2 copper layers, 0 parts

Commit message: complete redo with 32u4
Parts:
- added 16MHz1: 16mHz, Crystal:Crystal_SMD_3225-4Pin_3.2x2.5mm, F.Cu at (103.2, 79.4)
- added 22pF1: 22pF, Capacitor_SMD:C_0805_2012Metric, F.Cu at (107.9, 77.0)
- added 22pF2: 22pF, Capacitor_SMD:C_0805_2012Metric, F.Cu at (107.1, 79.4)
- added 500mA1: 500mA, Fuse:Fuse_1206_3216Metric, F.Cu at (73.2, 69.8)
- added C1: 1µF, Capacitor_SMD:C_0805_2012Metric, F.Cu at (84.1, 81.7)
- added C2: 0.1µF, Capacitor_SMD:C_0805_2012Metric, F.Cu at (104.0, 66.7)
- added C3: 0.1µF, Capacitor_SMD:C_0805_2012Metric, F.Cu at (104.0, 69.7)
- added C4: 0.1µF, Capacitor_SMD:C_0805_2012Metric, F.Cu at (104.0, 72.7)
- added C5: 10µF, Capacitor_SMD:C_0805_2012Metric, F.Cu at (104.0, 75.4)
- added D1: D_Small, Diode_SMD:D_SOD-123, B.Cu at (81.7, 32.5)
- added D2: D_Small, Diode_SMD:D_SOD-123, B.Cu at (100.8, 32.5)
- added D3: D_Small, Diode_SMD:D_SOD-123, B.Cu at (119.8, 32.5)
- added D4: D_Small, Diode_SMD:D_SOD-123, B.Cu at (81.8, 51.6)
- added D5: D_Small, Diode_SMD:D_SOD-123, B.Cu at (100.8, 51.6)
- added D6: D_Small, Diode_SMD:D_SOD-123, B.Cu at (119.9, 51.6)
- added K1: M, MX_Only:MXOnly-1U, F.Cu at (72.2, 35.7)
- added K2: A, MX_Only:MXOnly-1U-NoLED, F.Cu at (91.3, 35.7)
- added K3: X, MX_Only:MXOnly-1U-NoLED, F.Cu at (110.3, 35.7)
- added K4: P, MX_Only:MXOnly-1U-NoLED, F.Cu at (72.2, 54.8)
- added K5: C, MX_Only:MXOnly-1U-NoLED, F.Cu at (91.3, 54.8)
- added K6: B, MX_Only:MXOnly-1U-NoLED, F.Cu at (110.3, 54.8)
- added MaxCHIP32u4: ATmega32U4-A, Package_QFP:TQFP-44_10x10mm_P0.8mm, F.Cu at (91.6, 75.8)
- added MaxUSB-C: Molex-0548190589, random-keyboard-parts:Molex-0548190589, F.Cu at (63.8, 73.5)
- added R1: 10kΩ, Resistor_SMD:R_0805_2012Metric, F.Cu at (97.5, 65.9)
- added R2: 22Ω, Resistor_SMD:R_0805_2012Metric, F.Cu at (72.9, 74.6)
- added R3: 22Ω, Resistor_SMD:R_0805_2012Metric, F.Cu at (72.9, 72.2)
- added R4: 10kΩ, Resistor_SMD:R_0805_2012Metric, F.Cu at (88.9, 85.7)
- added ResetButton1: Reset Button, random-keyboard-parts:SKQG-1155865, F.Cu at (114.3, 81.0)
Routing:
- net GND: track 0.00 -> 111.1 mm, vias 0 -> 4
- net Row1: track 0.00 -> 87.5 mm, vias 0 -> 1
- net +5V: track 0.00 -> 80.9 mm, vias 0 -> 2
- net Row2: track 0.00 -> 64.7 mm, vias 0 -> 1
- net Col1: track 0.00 -> 48.8 mm
- net Col3: track 0.00 -> 45.4 mm
- net Col2: track 0.00 -> 37.9 mm
- net Net-(MaxCHIP32u4-~{RESET}): track 0.00 -> 31.4 mm
- net unconnected-(USB1-SHIELD-Pad6): track 0.00 -> 26.0 mm
- net Net-(MaxCHIP32u4-XTAL1): track 0.00 -> 15.2 mm
- net Net-(MaxCHIP32u4-D+): track 0.00 -> 14.8 mm
- net Net-(MaxCHIP32u4-D-): track 0.00 -> 14.8 mm
- net Net-(MaxCHIP32u4-XTAL2): track 0.00 -> 13.4 mm, vias 0 -> 2
- net Net-(D4-A): track 0.00 -> 7.18 mm
- net Net-(D5-A): track 0.00 -> 7.10 mm
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- added copper zone on B.Cu, net (none)
- added copper zone on F.Cu, net (none)
Other:
- board outline added: 60.3 x 62.7 mm
- board text added: "____ ____"
- board text added: "designed by max prime made in china"
- board text added: "maxpcb"
- board text added: "v1"
